File: hw/kicad/untitled.kicad_sch (KiCad schematic)
At the start: 64 parts

Commit message: mcu
Parts:
- C1, C3, C8: renamed from C?; footprint (none) -> Capacitor_SMD:C_0603_1608Metric
- C10, C11, C13, C14, C16, C17, C19, C20, C4, C5, C6, C9: renamed from C?; footprint (none) -> Capacitor_SMD:C_0805_2012Metric
- FB1, FB2: renamed from FB?; footprint (none) -> Capacitor_SMD:C_0603_1608Metric
- R1, R10, R11, R2, R3, R4, R5, R6, R7, R8, R9: renamed from R?; footprint (none) -> Resistor_SMD:R_0603_1608Metric
- gave numbers to parts that had none: 32
